File: TRI-Pcb/Mono-Test-Pcb.kicad_pcb (KiCad board)
At the start: 2 copper layers, 22 parts, among them J1 AudioJack4_Ground, J2 AudioJack4_Ground, J3 AudioJack4_Ground, U1 ESP32-C6-DevKitM-1

Commit message: versao 2 com correcao da orientacao dos sensores de tensao
Parts:
- moved OUT2 8.33 mm to (187.1, 39.2), turned to 180 degrees
- moved OUT3 8.01 mm to (221.4, 39.4), turned to 180 degrees
- moved OUT1 7.26 mm to (175.1, 95.3), turned to 0 degrees
Routing:
- net /3v3: track 224.1 -> 218.4 mm
- net /GPIO4: track 21.9 -> 18.8 mm
- net /GPIO2: track 12.6 -> 14.4 mm
